File: pcb/pica40.kicad_pcb (KiCad board)
At the start: 2 copper layers, 135 x 93.7 mm, 63 parts, among them SW1 SW_PUSH, SW10 SW_PUSH, SW11 SW_PUSH, SW12 SW_PUSH, SW13 SW_PUSH, SW14 SW_PUSH, SW15 SW_PUSH, SW16 SW_PUSH, SW17 SW_PUSH, SW18 SW_PUSH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

Commit message: fixes
Parts:
- D1, D10, D11, D12, D13, D14, D15, D16, D17, D18, D19, D2, D20, D3, D4, D5, D6, D7, D8, D9: footprint pica:D_SOD123 -> pica:D3_SMD
- LED1: footprint keebio:SK6812-MINI-E -> pica:SK6812-MINI-E; moved to F.Cu
- RE1: footprint keebio:RotaryEncoder_EC11-no-legs -> pica:RotaryEncoder_EC11-no-legs
- moved LED1 3.35 mm to (193.0, 99.0), turned to 0 degrees
Connections:
- LED1 pad 1: GND -> VCC
- LED1 pad 3: VCC -> GND
Routing:
- net LED: track 59.4 -> 42.8 mm, vias 0 -> 1
- net col2: track 193.6 -> 197.7 mm
- net VCC: track 50.3 -> 46.2 mm, vias 1 -> 2
- net row7: track 34.8 -> 36.7 mm
- net col1: track 285.5 -> 286.8 mm
- net BATT: track 80.6 -> 81.8 mm
- net row3: track 197.1 -> 197.8 mm, vias 0 -> 5
- net col3: track 142.0 -> 141.4 mm
- net GND: track 3.49 -> 3.99 mm
- net Net-(D18-Pad2): track 22.1 -> 21.7 mm, vias 1 -> 2
- net Net-(D10-Pad2): track 22.2 -> 21.8 mm, vias 1 -> 2
- net Net-(D4-Pad2): track 21.5 -> 21.2 mm, vias 1 -> 2
- net row0: track 99.2 -> 98.9 mm, vias 0 -> 5
- net Net-(D9-Pad2): track 21.9 -> 21.7 mm, vias 1 -> 2
- net row1: track 94.6 -> 94.4 mm, vias 0 -> 5
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