File: pcb/right.kicad_sch (KiCad schematic)
At the start: 49 parts, among them SW1 SW_PUSH, SW10 SW_PUSH, SW11 SW_PUSH, SW12 SW_PUSH, SW13 SW_PUSH, SW14 SW_PUSH, SW15 SW_PUSH, SW16 SW_PUSH, SW17 SW_PUSH, SW18 SW_PUSH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

Commit message: update cases, extra hole on right side
Parts:
- added H8: MountingHole, kbd:M2_HOLE_v2, symbol Mechanical:MountingHole
Changed lines of the file:
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@@
     (pin "2")
+  )
+  (symbol (lib_id "Mechanical:MountingHole") (at 237.49 142.24 0) (unit 1)
+    (in_bom yes) (on_board yes) (fields_autoplaced)
+    (property "Reference" "H8" (id 0) (at 240.03 140.9699 0)
+      (effects (font (size 1.27 1.27)) (justify left))
+    )
+    (property "Value" "MountingHole" (id 1) (at 240.03 143.5099 0)
+      (effects (font (size 1.27 1.27)) (justify left))
+    )
+    (property "Footprint" "kbd:M2_HOLE_v2" (id 2) (at 237.49 142.24 0)
+      (effects (font (size 1.27 1.27)) hide)
+    )
+    (property "Datasheet" "~" (id 3) (at 237.49 142.24 0)
+      (effects (font (size 1.27 1.27)) hide)
+    )
   )
   (symbol (lib_id "kbd:SW_PUSH") (at 143.51 111.76 0) (unit 1)
@@
       (reference "H7") (unit 1) (value "MountingHole") (footprint "kbd:M2_Hole_TH")
     )
+    (path "/b3f2c6fd-77d7-4bfe-862c-ca2878aef6b5"
+      (reference "H8") (unit 1) (value "MountingHole") (footprint "kbd:M2_HOLE_v2")
+    )
     (path "/050abe7e-8da5-4967-b5a8-32b5766f8192"
