File: pcb/right.kicad_sch (KiCad schematic)
At the start: 65 parts, among them SW1 SW_PUSH, SW10 SW_PUSH, SW11 SW_PUSH, SW12 SW_PUSH, SW13 SW_PUSH, SW14 SW_PUSH, SW15 SW_PUSH, SW16 SW_PUSH, SW17 SW_PUSH, SW18 SW_PUSH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

Commit message: non-reversible pcbs
Parts:
- removed BATTCONN1: Conn_01x02_Female, Connector_JST:JST_XH_S2B-XH-A_1x02_P2.50mm_Horizontal, symbol Connector:Conn_01x02_Female
- removed BATTSW1, BATTSW2: SW_SPDT, Button_Switch_SMD:SW_SPDT_PCM12, symbol Switch:SW_SPDT
- removed JP1, JP2, JP3, JP4, JP5, JP6, JP7, JP8: SolderJumper_2_Open, Jumper:SolderJumper-2_P1.3mm_Open_TrianglePad1.0x1.5mm, symbol Jumper:SolderJumper_2_Open
- removed LED1: YS-SK6812MINI-E, pica:SK6812-MINI-E, symbol kbd:YS-SK6812MINI-E
- removed OLED1: OLED, kbd:OLED_v2, symbol kbd:OLED
- removed RESET1: SW_Push, kbd:ResetSW, symbol Switch:SW_Push
- removed U1: ProMicro, keebio:ArduinoProMicro, symbol kbd:ProMicro
- removed USB1: HRO-TYPE-C-31-M-12, typec:HRO-TYPE-C-31-M-12-HandSoldering, symbol typec:HRO-TYPE-C-31-M-12
- added H8: MountingHole, kbd:M2_HOLE_v2, symbol Mechanical:MountingHole
- renumbered USB2 to USB1
Connections:
- net row0 is gone; now on net row7: D1.1 (K), D2.1 (K), D3.1 (K), D4.1 (K), D5.1 (K)
- net row1 is gone; now on net row6: D10.1 (K), D6.1 (K), D7.1 (K), D8.1 (K), D9.1 (K)
- net row2 is gone; now on net row5: D11.1 (K), D12.1 (K), D13.1 (K), D14.1 (K), D15.1 (K)
- net row3 is gone; now on net row4: D16.1 (K), D17.1 (K), D18.1 (K), D19.1 (K), D20.1 (K)
- no-connect marks 7 -> 3
Other:
- moved on the sheet: USB1

Commit message: v2
Parts:
- removed H8: MountingHole, kbd:M2_HOLE_v2, symbol Mechanical:MountingHole
- added BATTCONN1, BATTCONN2: Conn_01x02_Female, pica:JST_PH_S2B-PH-K_1x02_P2.00mm, symbol Connector:Conn_01x02_Female
- added BATTSW1: SW_SPDT, Button_Switch_SMD:SW_SPDT_PCM12, symbol Switch:SW_SPDT
- added JP1, JP2: SolderJumper_2_Open, Jumper:SolderJumper-2_P1.3mm_Open_TrianglePad1.0x1.5mm, symbol Jumper:SolderJumper_2_Open
- added RE2: RotaryEncoder_Switch, pica:RotaryEncoder_EC11, symbol Device:RotaryEncoder_Switch
- added U1: xiao-ble, pica:xiao-ble-tht, symbol kleeb-mcu:xiao-ble
- H1, H2, H3, H4, H5: footprint kbd:M2_HOLE_v2 -> pica:spacer_m2_3.4
- H6, H7: footprint kbd:M2_Hole_TH -> kbd:thread_m2
- RE1: footprint pica:RotaryEncoder_EC11-no-legs -> pica:RotaryEncoder_EC11
- SW1, SW10, SW11, SW12, SW13, SW14, SW15, SW16, SW17, SW18, SW19, SW2, SW3, SW4, SW5, SW6, SW7, SW8, SW9: footprint pica:CherryMX_Hotswap -> pica:CherryMX_Hotswap_ChocV2
- SW20: footprint pica:CherryMX_Hotswap_1.5 -> pica:CherryMX_Hotswap_ChocV2_1.5
- USB1: footprint typec:HRO-TYPE-C-31-M-12-HandSoldering -> pica:HRO-TYPE-C-31-M-12-data
Connections:
- net ENCA renamed ENCA_r
- net ENCA_r: now also JP1.1 (A), RE2.A; no longer USB1.11 (VBUS)
- net ENCB renamed ENCB_r
- net ENCB_r: now also USB1.5 (DN2), USB1.7 (DN1), RE2.B, U1.6 (A9_SCL/0.05_H); no longer USB1.12 (GND)
- net GND renamed GNDA
- net GNDA: now also USB1.12 (GND), BATTCONN1.2 (Pin_2), BATTCONN2.2 (Pin_2), RE2.C, U1.13 (GND), U1.18 (GND), U1.20 (GND)
- net col0 renamed col0_r
- net col0_r: now also U1.1 (A2/0.02_H); no longer USB1.10 (CC2)
- net col1 renamed col1_r
- net col1_r: now also U1.2 (A4/0.03_H); no longer USB1.9 (SBU1)
- net col2 renamed col2_r
- net col2_r: now also U1.3 (A10/0.28); no longer USB1.8 (DP2)
- net col3 renamed col3_r
- net col3_r: now also U1.4 (A11/0.29); no longer USB1.7 (DN1)
- net col4 renamed col4_r
- net col4_r: now also U1.5 (A8_SDA/0.04_H); no longer USB1.6 (DP1)
- net row4 renamed row3_r
- net row3_r: now also U1.8 (B9_RX/1.12); no longer USB1.5 (DN2)
- net row5 renamed row2_r
- net row2_r: now also U1.9 (A7_SCK/1.13); no longer USB1.4 (CC1)
- net row6 renamed row1_r
- net row1_r: now also U1.10 (A5_MISO/1.14); no longer USB1.3 (SBU2)
- net row7 renamed row0_r
- net row0_r: now also U1.11 (A6_MOSI/1.15); no longer USB1.2 (VBUS)
- new net: JP1.2 (B), JP2.2 (B), U1.7 (B8_TX/1.11)
- new net BATT_r: BATTCONN1.1 (Pin_1), BATTCONN2.1 (Pin_1), BATTSW1.2 (B)
- new net DATA_r: JP2.1 (A), USB1.6 (DP1), USB1.8 (DP2)
- new net RAW_r: BATTSW1.1 (A), U1.19 (BAT)
- new net VDD: U1.12 (3V3), USB1.11 (VBUS), USB1.2 (VBUS)
- no-connect marks 3 -> 16

Commit message: remove second encoder
Parts:
- removed RE2: RotaryEncoder_Switch, pica:RotaryEncoder_EC11, symbol Device:RotaryEncoder_Switch
Connections:
- no-connect marks 16 -> 14
Changed lines of the file:
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@@
   )
   (no_connect (at 156.21 48.26))
-  (no_connect (at 205.74 149.86))
   (no_connect (at 205.74 130.81))
   (no_connect (at 76.2 22.86))
@@
   (no_connect (at 78.74 54.61))
   (no_connect (at 156.21 33.02))
-  (no_connect (at 205.74 144.78))
   (no_connect (at 156.21 55.88))
   (no_connect (at 195.58 78.74))
@@
     (stroke (width 0) (type default) (color 0 0 0 0))
   )
-  (wire (pts (xy 190.5 147.32) (xy 179.07 147.32))
-    (stroke (width 0) (type default) (color 0 0 0 0))
-  )
   (wire (pts (xy 73.66 54.61) (xy 73.66 60.96))
     (stroke (width 0) (type default) (color 0 0 0 0))
@@
     )
   )
-  (global_label "ENCA_r" (shape input) (at 190.5 144.78 180) (fields_autoplaced)
-    (effects (font (size 1.27 1.27)) (justify right))
-    (property "Intersheet References" "${INTERSHEET_REFS}" (id 0) (at 181.495 144.7006 0)
-      (effects (font (size 1.27 1.27)) (justify right) hide)
-    )
-  )
   (global_label "ENCB_r" (shape input) (at 156.21 35.56 0) (fields_autoplaced)
     (effects (font (size 1.27 1.27)) (justify left))
@@
     (property "Intersheet References" "${INTERSHEET_REFS}" (id 0) (at 123.1106 70.4607 90)
       (effects (font (size 1.27 1.27)) (justify left) hide)
-    )
-  )
-  (global_label "ENCB_r" (shape input) (at 190.5 149.86 180) (fields_autoplaced)
-    (effects (font (size 1.27 1.27)) (justify right))
-    (property "Intersheet References" "${INTERSHEET_REFS}" (id 0) (at 181.3136 149.7806 0)
-      (effects (font (size 1.27 1.27)) (justify right) hide)
     )
   )
@@
     (pin "2")
   )
-  (symbol (lib_id "power:GNDA") (at 179.07 147.32 0) (unit 1)
-    (in_bom yes) (on_board yes)
-    (property "Reference" "#PWR012" (id 0) (at 179.07 153.67 0)
-      (effects (font (size 1.27 1.27)) hide)
-    )
-    (property "Value" "GNDA" (id 1) (at 175.26 148.59 0))
-    (property "Footprint" "" (id 2) (at 179.07 147.32 0)
-      (effects (font (size 1.27 1.27)) hide)
-    )
-    (property "Datasheet" "" (id 3) (at 179.07 147.32 0)
-      (effects (font (size 1.27 1.27)) hide)
-    )
-    (pin "1")
-  )
   (symbol (lib_id "Jumper:SolderJumper_2_Open") (at 45.72 49.53 0) (unit 1)
     (in_bom yes) (on_board yes)
@@
     (pin "2")
   )
-  (symbol (lib_id "Device:RotaryEncoder_Switch") (at 198.12 147.32 0) (unit 1)
-    (in_bom yes) (on_board yes) (fields_autoplaced)
-    (property "Reference" "RE2" (id 0) (at 198.12 137.16 0))
-    (property "Value" "RotaryEncoder_Switch" (id 1) (at 198.12 139.7 0))
-    (property "Footprint" "pica:RotaryEncoder_EC11" (id 2) (at 194.31 143.256 0)
-      (effects (font (size 1.27 1.27)) hide)
-    )
-    (property "Datasheet" "~" (id 3) (at 198.12 140.716 0)
-      (effects (font (size 1.27 1.27)) hide)
-    )
-    (pin "A")
-    (pin "B")
-    (pin "C")
-    (pin "S1")
-    (pin "S2")
-  )
   (symbol (lib_id "kbd:SW_PUSH") (at 95.25 111.76 0) (unit 1)
     (in_bom yes) (on_board yes) (fields_autoplaced)
@@
       (reference "#PWR011") (unit 1) (value "GNDA") (footprint "")
     )
-    (path "/6c4ed4f5-7c35-497f-a2f3-806f87f93da2"
-      (reference "#PWR012") (unit 1) (value "GNDA") (footprint "")
-    )
     (path "/13a73c69-55fd-483e-bf2e-5a7d5684ba95"
       (reference "BATTCONN1") (unit 1) (value "Conn_01x02_Female") (footprint "pica:JST_PH_S2B-PH-K_1x02_P2.00mm")
@@
       (reference "RE1") (unit 1) (value "RotaryEncoder_Switch") (footprint "pica:RotaryEncoder_EC11")
     )
-    (path "/e72527a5-82ee-4d5e-b649-b414d5533203"
-      (reference "RE2") (unit 1) (value "RotaryEncoder_Switch") (footprint "pica:RotaryEncoder_EC11")
-    )
     (path "/823ac192-cbf7-4f68-8620-7b19531db055"

Commit message: udpate pcb, remove unused files
Parts:
- removed BATTCONN1, BATTCONN2: Conn_01x02_Female, pica:JST_PH_S2B-PH-K_1x02_P2.00mm, symbol Connector:Conn_01x02_Female
- removed BATTSW1: SW_SPDT, Button_Switch_SMD:SW_SPDT_PCM12, symbol Switch:SW_SPDT
- removed D1, D10, D11, D12, D13, D14, D15, D16, D17, D18, D19, D2, D20, D3, D4, D5, D6, D7, D8, D9: D_Small, pica:D3_SMD, symbol Device:D_Small
- removed H1, H2, H3, H4, H5: MountingHole, pica:spacer_m2_3.4, symbol Mechanical:MountingHole
- removed H6, H7: MountingHole, kbd:thread_m2, symbol Mechanical:MountingHole
- removed JP1, JP2: SolderJumper_2_Open, Jumper:SolderJumper-2_P1.3mm_Open_TrianglePad1.0x1.5mm, symbol Jumper:SolderJumper_2_Open
- removed RE1: RotaryEncoder_Switch, pica:RotaryEncoder_EC11, symbol Device:RotaryEncoder_Switch
- removed SW1, SW10, SW11, SW12, SW13, SW14, SW15, SW16, SW17, SW18, SW19, SW2, SW3, SW4, SW5, SW6, SW7, SW8, SW9: SW_PUSH, pica:CherryMX_Hotswap_ChocV2, symbol kbd:SW_PUSH
- removed SW20: SW_PUSH, pica:CherryMX_Hotswap_ChocV2_1.5, symbol kbd:SW_PUSH
- removed U1: xiao-ble, pica:xiao-ble-tht, symbol kleeb-mcu:xiao-ble
- removed USB1: HRO-TYPE-C-31-M-12, pica:HRO-TYPE-C-31-M-12-data, symbol typec:HRO-TYPE-C-31-M-12
- added BATTCONN3, BATTCONN4: Conn_01x02_Female, pica:JST_PH_S2B-PH-K_1x02_P2.00mm, symbol Connector:Conn_01x02_Female
- added BATTSW2: SW_SPDT, Button_Switch_SMD:SW_SPDT_PCM12, symbol Switch:SW_SPDT
- added D21, D22, D23, D24, D25, D26, D27, D28, D29, D30, D31, D32, D33, D34, D35, D36, D37, D38, D39, D40: D_Small, pica:D3_SMD, symbol Device:D_Small
- added H10, H11, H12, H8, H9: MountingHole, pica:spacer_m2_3.4, symbol Mechanical:MountingHole
- added H13, H14: MountingHole, kbd:thread_m2, symbol Mechanical:MountingHole
- added J2: MJ-4PP-9, pica:MJ-4PP-9_1side, symbol kbd:MJ-4PP-9
- added JP4, JP5, JP6: SolderJumper_2_Open, Jumper:SolderJumper-2_P1.3mm_Open_TrianglePad1.0x1.5mm, symbol Jumper:SolderJumper_2_Open
- added RE2: RotaryEncoder_Switch, pica:RotaryEncoder_EC11, symbol Device:RotaryEncoder_Switch
- added SW21, SW22, SW23, SW24, SW25, SW26, SW27, SW28, SW29, SW30, SW31, SW32, SW33, SW34, SW35, SW36, SW37, SW38, SW39: SW_PUSH, pica:CherryMX_Hotswap_ChocV2, symbol kbd:SW_PUSH
- added SW40: SW_PUSH, pica:CherryMX_Hotswap_ChocV2_1.5, symbol kbd:SW_PUSH
- added U2: xiao-ble, pica:xiao-ble-tht, symbol kleeb-mcu:xiao-ble
- added USB2: HRO-TYPE-C-31-M-12, pica:HRO-TYPE-C-31-M-12-data, symbol typec:HRO-TYPE-C-31-M-12
Connections:
- net BATT_r: now also BATTCONN3.1 (Pin_1), BATTCONN4.1 (Pin_1), BATTSW2.2 (B)
- net DATA_r: now also J2.A, JP6.1 (A), USB2.6 (DP1), USB2.8 (DP2)
- net ENCA_r: now also JP4.2 (B), RE2.A, U2.6 (A9_SCL/0.05_H)
- net ENCB_r: now also J2.B, JP4.1 (A), JP5.1 (A), RE2.B, USB2.5 (DN2), USB2.7 (DN1)
- net GNDA: now also BATTCONN3.2 (Pin_2), BATTCONN4.2 (Pin_2), J2.C, RE2.C, U2.13 (GND), U2.18 (GND), U2.20 (GND), USB2.1 (GND), USB2.12 (GND)
- net RAW_r: now also BATTSW2.1 (A), U2.19 (BAT)
- net VDD: now also J2.D, U2.12 (3V3), USB2.11 (VBUS), USB2.2 (VBUS)
- net col0_r: now also SW21.2, SW26.2, SW31.2, SW36.2, U2.1 (A2/0.02_H)
- net col1_r: now also SW22.2, SW27.2, SW32.2, SW37.2, U2.2 (A4/0.03_H)
- net col2_r: now also SW23.2, SW28.2, SW33.2, SW38.2, U2.3 (A10/0.28)
- net col3_r: now also SW24.2, SW29.2, SW34.2, SW39.2, U2.4 (A11/0.29)
- net col4_r: now also SW25.2, SW30.2, SW35.2, SW40.2, U2.5 (A8_SDA/0.04_H)
- net row0_r: now also D21.1 (K), D22.1 (K), D23.1 (K), D24.1 (K), D25.1 (K), U2.11 (A6_MOSI/1.15)
- net row1_r: now also D26.1 (K), D27.1 (K), D28.1 (K), D29.1 (K), D30.1 (K), U2.10 (A5_MISO/1.14)
- net row2_r: now also D31.1 (K), D32.1 (K), D33.1 (K), D34.1 (K), D35.1 (K), U2.9 (A7_SCK/1.13)
- net row3_r: now also D36.1 (K), D37.1 (K), D38.1 (K), D39.1 (K), D40.1 (K), U2.8 (B9_RX/1.12)
- new net: D26.2 (A), SW26.1
- new net: D24.2 (A), SW24.1
- new net: D27.2 (A), SW27.1
- new net: JP5.2 (B), JP6.2 (B), U2.7 (B8_TX/1.11)
- new net: D30.2 (A), SW30.1
- new net: D35.2 (A), SW35.1
- new net: D28.2 (A), SW28.1
- new net: D37.2 (A), SW37.1
- new net: D29.2 (A), SW29.1
- new net: D33.2 (A), SW33.1
- new net: D23.2 (A), SW23.1
- new net: D32.2 (A), SW32.1
- new net: D36.2 (A), SW36.1
- new net: D22.2 (A), SW22.1
- new net: D34.2 (A), SW34.1
- new net: D40.2 (A), SW40.1
- new net: D21.2 (A), SW21.1
- new net: D38.2 (A), SW38.1
- new net: D25.2 (A), SW25.1
- new net: D39.2 (A), SW39.1
- new net: D31.2 (A), SW31.1
