File: pcb/left.kicad_pcb (KiCad board)
At the start: 2 copper layers, 135 x 95.7 mm, 56 parts, among them SW1 SW_PUSH, SW10 SW_PUSH, SW11 SW_PUSH, SW12 SW_PUSH, SW13 SW_PUSH, SW14 SW_PUSH, SW15 SW_PUSH, SW16 SW_PUSH, SW17 SW_PUSH, SW18 SW_PUSH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

Commit message: fix battery connector footprint
Parts:
- BATTCONN1: footprint Connector_JST:JST_XH_S2B-XH-A_1x02_P2.50mm_Horizontal -> Connector_JST:JST_PH_S2B-PH-K_1x02_P2.00mm_Horizontal
- moved BATTCONN1 0.80 mm to (197.5, 96.0)
Changed lines of the file:
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@@
     )
   )
-  (footprint "Connector_JST:JST_XH_S2B-XH-A_1x02_P2.50mm_Horizontal" (layer "F.Cu")
-    (at 196.7 96 -90)
-    (descr "JST XH series connector, S2B-XH-A (http://www.jst-mfg.com/product/pdf/eng/eXH.pdf), generated with kicad-footprint-generator")
-    (tags "connector JST XH horizontal")
+  (footprint "Connector_JST:JST_PH_S2B-PH-K_1x02_P2.00mm_Horizontal" (layer "F.Cu")
+    (at 197.5 96 -90)
+    (descr "JST PH series connector, S2B-PH-K (http://www.jst-mfg.com/product/pdf/eng/ePH.pdf), generated with kicad-footprint-generator")
+    (tags "connector JST PH top entry")
     (property "Sheetfile" "left.kicad_sch")
     (property "Sheetname" "")
     (attr through_hole)
-    (fp_text reference "BATTCONN1" (at 1.25 -3.5 -90) (layer "F.SilkS") hide
+    (fp_text reference "BATTCONN1" (at 1 -2.55 -90) (layer "F.SilkS") hide
       (effects (font (size 1 1) (thickness 0.15)))
     )
-    (fp_text value "Conn_01x02_Female" (at 1.25 10.4 -90) (layer "F.Fab")
+    (fp_text value "Conn_01x02_Female" (at 1 7.45 -90) (layer "F.Fab")
       (effects (font (size 1 1) (thickness 0.15)))
     )
-    (fp_text user "${REFERENCE}" (at 1.25 3.45 -90) (layer "F.Fab")
+    (fp_text user "${REFERENCE}" (at 1 2.5 -90) (layer "F.Fab")
       (effects (font (size 1 1) (thickness 0.15)))
     )
-    (fp_line (start -0.3 -2.1) (end 0.3 -2.1) (layer "F.SilkS") (width 0.12))
-    (fp_line (start 2.75 3.2) (end 2.25 3.2) (layer "F.SilkS") (width 0.12))
-    (fp_line (start -0.25 8.7) (end 0.25 8.7) (layer "F.SilkS") (width 0.12))
-    (fp_line (start 0.25 8.7) (end 0.25 3.2) (layer "F.SilkS") (width 0.12))
-    (fp_line (start -1.14 -2.41) (end -1.14 2.09) (layer "F.SilkS") (width 0.12))
-    (fp_line (start 0 -1.5) (end -0.3 -2.1) (layer "F.SilkS") (width 0.12))
-    (fp_line (start 3.64 -2.41) (end 3.64 2.09) (layer "F.SilkS") (width 0.12))
-    (fp_line (start 3.64 2.09) (end 1.25 2.09) (layer "F.SilkS") (width 0.12))
-    (fp_line (start -2.56 9.31) (end -2.56 -2.41) (layer "F.SilkS") (width 0.12))
-    (fp_line (start 2.75 8.7) (end 2.75 3.2) (layer "F.SilkS") (width 0.12))
-    (fp_line (start 5.06 -2.41) (end 3.64 -2.41) (layer "F.SilkS") (width 0.12))
-    (fp_line (start -2.56 -2.41) (end -1.14 -2.41) (layer "F.SilkS") (width 0.12))
-    (fp_line (start 1.25 9.31) (end 5.06 9.31) (layer "F.SilkS") (width 0.12))
-    (fp_line (start -1.14 2.09) (end 1.25 2.09) (layer "F.SilkS") (width 0.12))
-    (fp_line (start 0.25 3.2) (end -0.25 3.2) (layer "F.SilkS") (width 0.12))
-    (fp_line (start 5.06 9.31) (end 5.06 -2.41) (layer "F.SilkS") (width 0.12))
-    (fp_line (start 0.3 -2.1) (end 0 -1.5) (layer "F.SilkS") (width 0.12))
-    (fp_line (start 1.25 9.31) (end -2.56 9.31) (layer "F.SilkS") (width 0.12))
-    (fp_line (start 2.25 8.7) (end 2.75 8.7) (layer "F.SilkS") (width 0.12))
-    (fp_line (start 2.25 3.2) (end 2.25 8.7) (layer "F.SilkS") (width 0.12))
-    (fp_line (start -0.25 3.2) (end -0.25 8.7) (layer "F.SilkS") (width 0.12))
-    (fp_line (start -2.95 9.7) (end 5.45 9.7) (layer "F.CrtYd") (width 0.05))
-    (fp_line (start 5.45 -2.8) (end -2.95 -2.8) (layer "F.CrtYd") (width 0.05))
-    (fp_line (start 5.45 9.7) (end 5.45 -2.8) (layer "F.CrtYd") (width 0.05))
-    (fp_line (start -2.95 -2.8) (end -2.95 9.7) (layer "F.CrtYd") (width 0.05))
-    (fp_line (start 1.25 9.2) (end -2.45 9.2) (layer "F.Fab") (width 0.1))
-    (fp_line (start 0 1.2) (end 0.625 2.2) (layer "F.Fab") (width 0.1))
-    (fp_line (start 3.75 -2.3) (end 3.75 2.2) (layer "F.Fab") (width 0.1))
-    (fp_line (start 1.25 9.2) (end 4.95 9.2) (layer "F.Fab") (width 0.1))
-    (fp_line (start -1.25 -2.3) (end -1.25 2.2) (layer "F.Fab") (width 0.1))
-    (fp_line (start -0.625 2.2) (end 0 1.2) (layer "F.Fab") (width 0.1))
-    (fp_line (start 3.75 2.2) (end 1.25 2.2) (layer "F.Fab") (width 0.1))
-    (fp_line (start -1.25 2.2) (end 1.25 2.2) (layer "F.Fab") (width 0.1))
-    (fp_line (start -2.45 -2.3) (end -1.25 -2.3) (layer "F.Fab") (width 0.1))
-    (fp_line (start 4.95 -2.3) (end 3.75 -2.3) (layer "F.Fab") (width 0.1))
-    (fp_line (start -2.45 9.2) (end -2.45 -2.3) (layer "F.Fab") (width 0.1))
-    (fp_line (start 4.95 9.2) (end 4.95 -2.3) (layer "F.Fab") (width 0.1))
-    (pad "1" thru_hole roundrect (at 0 0 270) (size 1.7 2) (drill 1) (layers *.Cu "B.Mask") (roundrect_rratio 0.1470588235)
+    (fp_line (start 4.06 0.14) (end 3.14 0.14) (layer "F.SilkS") (width 0.12))
+    (fp_line (start -1.3 4.1) (end -0.3 4.1) (layer "F.SilkS") (width 0.12))
+    (fp_line (start 4.06 -1.46) (end 3.14 -1.46) (layer "F.SilkS") (width 0.12))
+    (fp_line (start -0.86 0.14) (end -1.14 0.14) (layer "F.SilkS") (width 0.12))
+    (fp_line (start 2.3 2.5) (end 3.3 2.5) (layer "F.SilkS") (width 0.12))
+    (fp_line (start -0.86 0.14) (end -0.86 -1.075) (layer "F.SilkS") (width 0.12))
+    (fp_line (start -1.14 -1.46) (end -2.06 -1.46) (layer "F.SilkS") (width 0.12))
+    (fp_line (start 3.14 -1.46) (end 3.14 0.14) (layer "F.SilkS") (width 0.12))
+    (fp_line (start 1.5 2) (end 1.5 6.36) (layer "F.SilkS") (width 0.12))
+    (fp_line (start -0.3 4.1) (end -0.3 6.36) (layer "F.SilkS") (width 0.12))
+    (fp_line (start -2.06 0.14) (end -1.14 0.14) (layer "F.SilkS") (width 0.12))
+    (fp_line (start 3.14 0.14) (end 2.86 0.14) (layer "F.SilkS") (width 0.12))
+    (fp_line (start -0.3 2.5) (end -1.3 2.5) (layer "F.SilkS") (width 0.12))
+    (fp_line (start 0.5 6.36) (end 0.5 2) (layer "F.SilkS") (width 0.12))
+    (fp_line (start -1.14 0.14) (end -1.14 -1.46) (layer "F.SilkS") (width 0.12))
+    (fp_line (start 2.3 4.1) (end 2.3 2.5) (layer "F.SilkS") (width 0.12))
+    (fp_line (start -2.06 6.36) (end 4.06 6.36) (layer "F.SilkS") (width 0.12))
+    (fp_line (start -1.3 2.5) (end -1.3 4.1) (layer "F.SilkS") (width 0.12))
+    (fp_line (start 3.3 4.1) (end 2.3 4.1) (layer "F.SilkS") (width 0.12))
+    (fp_line (start 0.5 2) (end 1.5 2) (layer "F.SilkS") (width 0.12))
+    (fp_line (start -0.8 4.1) (end -0.8 6.36) (layer "F.SilkS") (width 0.12))
+    (fp_line (start -2.06 -1.46) (end -2.06 6.36) (layer "F.SilkS") (width 0.12))
+    (fp_line (start -0.3 4.1) (end -0.3 2.5) (layer "F.SilkS") (width 0.12))
+    (fp_line (start 3.3 2.5) (end 3.3 4.1) (layer "F.SilkS") (width 0.12))
+    (fp_line (start 4.06 6.36) (end 4.06 -1.46) (layer "F.SilkS") (width 0.12))
+    (fp_line (start 4.45 -1.85) (end -2.45 -1.85) (layer "F.CrtYd") (width 0.05))
+    (fp_line (start -2.45 -1.85) (end -2.45 6.75) (layer "F.CrtYd") (width 0.05))
+    (fp_line (start -2.45 6.75) (end 4.45 6.75) (layer "F.CrtYd") (width 0.05))
+    (fp_line (start 4.45 6.75) (end 4.45 -1.85) (layer "F.CrtYd") (width 0.05))
+    (fp_line (start -1.95 -1.35) (end -1.95 6.25) (layer "F.Fab") (width 0.1))
+    (fp_line (start -0.5 1.375) (end 0.5 1.375) (layer "F.Fab") (width 0.1))
+    (fp_line (start 3.95 -1.35) (end 3.25 -1.35) (layer "F.Fab") (width 0.1))
+    (fp_line (start -1.95 6.25) (end 3.95 6.25) (layer "F.Fab") (width 0.1))
+    (fp_line (start 0 0.875) (end -0.5 1.375) (layer "F.Fab") (width 0.1))
+    (fp_line (start 3.25 -1.35) (end 3.25 0.25) (layer "F.Fab") (width 0.1))
+    (fp_line (start -1.25 0.25) (end -1.25 -1.35) (layer "F.Fab") (width 0.1))
+    (fp_line (start -1.25 -1.35) (end -1.95 -1.35) (layer "F.Fab") (width 0.1))
+    (fp_line (start 0.5 1.375) (end 0 0.875) (layer "F.Fab") (width 0.1))
+    (fp_line (start 3.95 6.25) (end 3.95 -1.35) (layer "F.Fab") (width 0.1))
+    (fp_line (start 3.25 0.25) (end -1.25 0.25) (layer "F.Fab") (width 0.1))
+    (pad "1" thru_hole roundrect (at 0 0 270) (size 1.2 1.75) (drill 0.75) (layers *.Cu "B.Mask") (roundrect_rratio 0.208333)
       (net 1 "BATT") (pinfunction "Pin_1") (pintype "passive"))
-    (pad "2" thru_hole oval (at 2.5 0 270) (size 1.7 2) (drill 1) (layers *.Cu "B.Mask")
+    (pad "2" thru_hole oval (at 2 0 270) (size 1.2 1.75) (drill 0.75) (layers *.Cu "B.Mask")
       (net 2 "GND") (pinfunction "Pin_2") (pintype "passive"))
-    (model "${KICAD6_3DMODEL_DIR}/Connector_JST.3dshapes/JST_XH_S2B-XH-A_1x02_P2.50mm_Horizontal.wrl"
+    (model "${KICAD6_3DMODEL_DIR}/Connector_JST.3dshapes/JST_PH_S2B-PH-K_1x02_P2.00mm_Horizontal.wrl"
       (offset (xyz 0 0 0))
       (scale (xyz 1 1 1))

Commit message: fix
Parts:
- moved BATTCONN1 0.75 mm to (196.8, 96.0)
Changed lines of the file:
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@@
   )
   (footprint "Connector_JST:JST_PH_S2B-PH-K_1x02_P2.00mm_Horizontal" (layer "F.Cu")
-    (at 197.5 96 -90)
+    (at 196.75 96 -90)
     (descr "JST PH series connector, S2B-PH-K (http://www.jst-mfg.com/product/pdf/eng/ePH.pdf), generated with kicad-footprint-generator")
     (tags "connector JST PH top entry")
@@
     (fp_line (start 3.95 6.25) (end 3.95 -1.35) (layer "F.Fab") (width 0.1))
     (fp_line (start 3.25 0.25) (end -1.25 0.25) (layer "F.Fab") (width 0.1))
-    (pad "1" thru_hole roundrect (at 0 0 270) (size 1.2 1.75) (drill 0.75) (layers *.Cu "B.Mask") (roundrect_rratio 0.208333)
+    (pad "1" thru_hole roundrect (at 0 0 270) (size 1.2 1.75) (drill 0.75) (layers *.Cu "B.Mask") (roundrect_rratio 0.2083333333)
       (net 1 "BATT") (pinfunction "Pin_1") (pintype "passive"))
     (pad "2" thru_hole oval (at 2 0 270) (size 1.2 1.75) (drill 0.75) (layers *.Cu "B.Mask")
