File: plate-cover/pica40.kicad_sch (KiCad schematic)
At the start: 25 parts, among them SW1 SW_PUSH, SW10 SW_PUSH, SW11 SW_PUSH, SW12 SW_PUSH, SW13 SW_PUSH, SW14 SW_PUSH, SW15 SW_PUSH, SW16 SW_PUSH, SW17 SW_PUSH, SW18 SW_PUSH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

Commit message: add breakaway plate, replace battery connector
Parts:
- added BR1: MountingHole, kbd:Breakaway_Tabs, symbol Mechanical:MountingHole
- added H6, H7: MountingHole, kbd:M2_Hole_TH, symbol Mechanical:MountingHole
- added RE1: RotaryEncoder_Switch, pica:EC11_Hole_Breakaway, symbol Device:RotaryEncoder_Switch
Connections:
- new net ENCA: RE1.A
- new net ENCB: RE1.B
- new net GND: RE1.C
- no-connect marks 0 -> 2
Changed lines of the file:
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@@
 (kicad_sch (version 20211123) (generator eeschema)
   (paper "A4")
+  (no_connect (at 203.2 153.67))
+  (no_connect (at 203.2 148.59))
   (wire (pts (xy 74.93 91.44) (xy 74.93 92.71))
     (stroke (width 0) (type default) (color 0 0 0 0))
@@
   (wire (pts (xy 74.93 132.08) (xy 74.93 133.35))
     (stroke (width 0) (type default) (color 0 0 0 0))
+  )
+  (wire (pts (xy 187.96 151.13) (xy 176.53 151.13))
+    (stroke (width 0) (type default) (color 0 0 0 0))
+  )
+  (global_label "ENCB" (shape input) (at 187.96 153.67 180) (fields_autoplaced)
+    (effects (font (size 1.27 1.27)) (justify right))
+    (property "Intersheet References" "${INTERSHEET_REFS}" (id 0) (at 180.5274 153.5906 0)
+      (effects (font (size 1.27 1.27)) (justify right) hide)
+    )
+  )
+  (global_label "ENCA" (shape input) (at 187.96 148.59 180) (fields_autoplaced)
+    (effects (font (size 1.27 1.27)) (justify right))
+    (property "Intersheet References" "${INTERSHEET_REFS}" (id 0) (at 180.7088 148.5106 0)
+      (effects (font (size 1.27 1.27)) (justify right) hide)
+    )
+  )
+  (symbol (lib_id "Device:RotaryEncoder_Switch") (at 195.58 151.13 0) (unit 1)
+    (in_bom yes) (on_board yes) (fields_autoplaced)
+    (property "Reference" "RE1" (id 0) (at 195.58 140.97 0))
+    (property "Value" "RotaryEncoder_Switch" (id 1) (at 195.58 143.51 0))
+    (property "Footprint" "pica:EC11_Hole_Breakaway" (id 2) (at 191.77 147.066 0)
+      (effects (font (size 1.27 1.27)) hide)
+    )
+    (property "Datasheet" "~" (id 3) (at 195.58 144.526 0)
+      (effects (font (size 1.27 1.27)) hide)
+    )
+    (pin "A")
+    (pin "B")
+    (pin "C")
+    (pin "S1")
+    (pin "S2")
   )
   (symbol (lib_id "kbd:SW_PUSH") (at 82.55 111.76 0) (unit 1)
@@
     )
   )
+  (symbol (lib_id "Mechanical:MountingHole") (at 237.49 158.75 0) (unit 1)
+    (in_bom yes) (on_board yes) (fields_autoplaced)
+    (property "Reference" "H7" (id 0) (at 240.03 157.4799 0)
+      (effects (font (size 1.27 1.27)) (justify left))
+    )
+    (property "Value" "MountingHole" (id 1) (at 240.03 160.0199 0)
+      (effects (font (size 1.27 1.27)) (justify left))
+    )
+    (property "Footprint" "kbd:M2_Hole_TH" (id 2) (at 237.49 158.75 0)
+      (effects (font (size 1.27 1.27)) hide)
+    )
+    (property "Datasheet" "~" (id 3) (at 237.49 158.75 0)
+      (effects (font (size 1.27 1.27)) hide)
+    )
+  )
   (symbol (lib_id "kbd:SW_PUSH") (at 62.23 91.44 0) (unit 1)
     (in_bom yes) (on_board yes) (fields_autoplaced)
@@
     (pin "2")
   )
+  (symbol (lib_id "power:GND") (at 176.53 151.13 0) (unit 1)
+    (in_bom yes) (on_board yes) (fields_autoplaced)
+    (property "Reference" "#PWR013" (id 0) (at 176.53 157.48 0)
+      (effects (font (size 1.27 1.27)) hide)
+    )
+    (property "Value" "GND" (id 1) (at 176.53 156.21 0))
+    (property "Footprint" "" (id 2) (at 176.53 151.13 0)
+      (effects (font (size 1.27 1.27)) hide)
+    )
+    (property "Datasheet" "" (id 3) (at 176.53 151.13 0)
+      (effects (font (size 1.27 1.27)) hide)
+    )
+    (pin "1")
+  )
+  (symbol (lib_id "Mechanical:MountingHole") (at 237.49 152.4 0) (unit 1)
+    (in_bom yes) (on_board yes) (fields_autoplaced)
+    (property "Reference" "H6" (id 0) (at 240.03 151.1299 0)
+      (effects (font (size 1.27 1.27)) (justify left))
+    )
+    (property "Value" "MountingHole" (id 1) (at 240.03 153.6699 0)
+      (effects (font (size 1.27 1.27)) (justify left))
+    )
+    (property "Footprint" "kbd:M2_Hole_TH" (id 2) (at 237.49 152.4 0)
+      (effects (font (size 1.27 1.27)) hide)
+    )
+    (property "Datasheet" "~" (id 3) (at 237.49 152.4 0)
+      (effects (font (size 1.27 1.27)) hide)
+    )
+  )
+  (symbol (lib_id "Mechanical:MountingHole") (at 194.31 92.71 0) (unit 1)
+    (in_bom yes) (on_board yes) (fields_autoplaced)
+    (property "Reference" "BR1" (id 0) (at 196.85 91.4399 0)
+      (effects (font (size 1.27 1.27)) (justify left))
+    )
+    (property "Value" "MountingHole" (id 1) (at 196.85 93.9799 0)
+      (effects (font (size 1.27 1.27)) (justify left))
+    )
+    (property "Footprint" "kbd:Breakaway_Tabs" (id 2) (at 194.31 92.71 0)
+      (effects (font (size 1.27 1.27)) hide)
+    )
+    (property "Datasheet" "~" (id 3) (at 194.31 92.71 0)
+      (effects (font (size 1.27 1.27)) hide)
+    )
+  )
   (symbol (lib_id "kbd:SW_PUSH") (at 143.51 91.44 0) (unit 1)
     (in_bom yes) (on_board yes) (fields_autoplaced)
@@
   )
   (symbol_instances
+    (path "/ed356ae0-d310-43a9-a1ad-70f09e4803a8"
+      (reference "#PWR013") (unit 1) (value "GND") (footprint "")
+    )
+    (path "/fb44414e-45b4-4fed-a80e-b6104c96abc3"
+      (reference "BR1") (unit 1) (value "MountingHole") (footprint "kbd:Breakaway_Tabs")
+    )
     (path "/a296e5d3-1285-4b08-bd6b-dfc91d480e82"
       (reference "H1") (unit 1) (value "MountingHole") (footprint "kbd:M2_Hole_TH")
@@
       (reference "H5") (unit 1) (value "MountingHole") (footprint "kbd:M2_Hole_TH")
     )
+    (path "/f52c0b43-7ef2-43de-9e7f-2633ce8cd351"
+      (reference "H6") (unit 1) (value "MountingHole") (footprint "kbd:M2_Hole_TH")
+    )
+    (path "/dc3229c7-5794-49f0-b14b-ffc46123b28f"
+      (reference "H7") (unit 1) (value "MountingHole") (footprint "kbd:M2_Hole_TH")
+    )
+    (path "/050abe7e-8da5-4967-b5a8-32b5766f8192"
+      (reference "RE1") (unit 1) (value "RotaryEncoder_Switch") (footprint "pica:EC11_Hole_Breakaway")
+    )
     (path "/dfe7bca9-eacf-484d-9fb9-819b1262f86e"
