File: case/cover-big-hole-acrylic.kicad_pcb (KiCad board)
At the start: 2 copper layers, 20.5 x 58.5 mm, 4 parts

Commit message: adjust top plate, add new cover in PCB style
Other:
- board size 20.5 x 58.5 mm -> 20.5 x 57.2 mm
Changed lines of the file:
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@@
   (gr_line (start 125.5 106) (end 125.5 60) (layer "Edge.Cuts") (width 0.1))
   (gr_arc (start 144.5 60) (mid 145.56066 60.43934) (end 146 61.5) (layer "Edge.Cuts") (width 0.1))
-  (gr_line (start 127 108.5) (end 143.75 118.25) (layer "Edge.Cuts") (width 0.1))
   (gr_arc (start 127 108.5) (mid 125.931823 107.440906) (end 125.5 106) (layer "Edge.Cuts") (width 0.1))
-  (gr_line (start 146 117) (end 146 61.5) (layer "Edge.Cuts") (width 0.1))
-  (gr_arc (start 146 117) (mid 145.251202 118.302163) (end 143.75 118.25) (layer "Edge.Cuts") (width 0.1))
+  (gr_line (start 146 114) (end 146 61.5) (layer "Edge.Cuts") (width 0.1))
+  (gr_circle (center 136 103.25) (end 136 99.25) (layer "Edge.Cuts") (width 0.1) (fill none))
+  (gr_arc (start 146 114) (mid 144.54209 116.680055) (end 141.5 116.912176) (layer "Edge.Cuts") (width 0.1))
   (gr_line (start 144.5 60) (end 125.5 60) (layer "Edge.Cuts") (width 0.1))
+  (gr_line (start 141.5 116.912176) (end 127 108.5) (layer "Edge.Cuts") (width 0.1))
 )

Commit message: fix DXF files for new covers
Other:
- board size 20.5 x 57.2 mm -> 20.5 x 58.5 mm
Changed lines of the file:
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@@
     (pad "" np_thru_hole circle locked (at 0 0) (size 2.3 2.3) (drill 2.3) (layers *.Cu *.Mask))
   )
+  (gr_arc (start 146 117) (mid 145.251221 118.302195) (end 143.75 118.25) (layer "Edge.Cuts") (width 0.1))
   (gr_line (start 125.5 106) (end 125.5 60) (layer "Edge.Cuts") (width 0.1))
   (gr_arc (start 144.5 60) (mid 145.56066 60.43934) (end 146 61.5) (layer "Edge.Cuts") (width 0.1))
+  (gr_line (start 127 108.5) (end 143.75 118.25) (layer "Edge.Cuts") (width 0.1))
   (gr_arc (start 127 108.5) (mid 125.931823 107.440906) (end 125.5 106) (layer "Edge.Cuts") (width 0.1))
-  (gr_line (start 146 114) (end 146 61.5) (layer "Edge.Cuts") (width 0.1))
+  (gr_line (start 146 117) (end 146 61.5) (layer "Edge.Cuts") (width 0.1))
   (gr_circle (center 136 103.25) (end 136 99.25) (layer "Edge.Cuts") (width 0.1) (fill none))
-  (gr_arc (start 146 114) (mid 144.54209 116.680055) (end 141.5 116.912176) (layer "Edge.Cuts") (width 0.1))
   (gr_line (start 144.5 60) (end 125.5 60) (layer "Edge.Cuts") (width 0.1))
-  (gr_line (start 141.5 116.912176) (end 127 108.5) (layer "Edge.Cuts") (width 0.1))
 )
