File: case/bottom-metal.kicad_pcb (KiCad board)
At the start: 2 copper layers, 137.8 x 95.7 mm, 7 parts

Commit message: fix dxf files
Parts:
- H1, H2, H3, H4, H5, H6, H7: footprint kbd:thread_m2 -> pica:thread_m2_hole
Changed lines of the file:
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@@
     (pad_to_mask_clearance 0)
     (pcbplotparams
-      (layerselection 0x0000080_7ffffffe)
+      (layerselection 0x0001000_7ffffffe)
       (disableapertmacros false)
       (usegerberextensions false)
@@
       (svguseinch false)
       (svgprecision 6)
-      (excludeedgelayer false)
+      (excludeedgelayer true)
       (plotframeref false)
       (viasonmask false)
@@
       (hpglpenspeed 20)
       (hpglpendiameter 15.000000)
-      (dxfpolygonmode true)
+      (dxfpolygonmode false)
       (dxfimperialunits false)
       (dxfusepcbnewfont true)
@@
   )
   (net 0 "")
-  (footprint "kbd:thread_m2" (layer "F.Cu")
+  (footprint "pica:thread_m2_hole" (layer "F.Cu")
     (at 215.25 86.5)
     (descr "Mounting Hole 2.2mm, no annular, M2")
@@
     (property "Sheetfile" "full.kicad_sch")
     (property "Sheetname" "")
-    (attr exclude_from_pos_files)
+    (attr exclude_from_pos_files exclude_from_bom)
     (fp_text reference "H7" (at -0.95 -0.55) (layer "F.Fab") hide
       (effects (font (size 1 1) (thickness 0.15)))
@@
       (effects (font (size 1 1) (thickness 0.15)))
     )
-    (pad "" np_thru_hole circle locked (at 0 0) (size 2.3 2.3) (drill 2.3) (layers *.Cu *.Mask))
+    (fp_circle (center 0 0) (end 1.15 0) (layer "Edge.Cuts") (width 0.1) (fill none))
   )
-  (footprint "kbd:thread_m2" (layer "F.Cu")
+  (footprint "pica:thread_m2_hole" (layer "F.Cu")
     (at 105.25 103.25 5)
     (descr "Mounting Hole 2.2mm, no annular, M2")
@@
       (effects (font (size 1 1) (thickness 0.15)))
     )
-    (pad "" np_thru_hole circle locked (at 0 0 5) (size 2.3 2.3) (drill 2.3) (layers *.Cu *.Mask))
+    (fp_circle (center 0 0) (end 1.15 0) (layer "Edge.Cuts") (width 0.1) (fill none))
   )
-  (footprint "kbd:thread_m2" (layer "F.Cu")
+  (footprint "pica:thread_m2_hole" (layer "F.Cu")
     (at 124.8 77)
     (descr "Mounting Hole 2.2mm, no annular, M2")
@@
       (effects (font (size 1 1) (thickness 0.15)))
     )
-    (pad "" np_thru_hole circle locked (at 0 0) (size 2.3 2.3) (drill 2.3) (layers *.Cu *.Mask))
+    (fp_circle (center 0 0) (end 1.15 0) (layer "Edge.Cuts") (width 0.1) (fill none))
   )
-  (footprint "kbd:thread_m2" (layer "F.Cu")
+  (footprint "pica:thread_m2_hole" (layer "F.Cu")
     (at 184 79.5)
     (descr "Mounting Hole 2.2mm, no annular, M2")
@@
       (effects (font (size 1 1) (thickness 0.15)))
     )
-    (pad "" np_thru_hole circle locked (at 0 0) (size 2.3 2.3) (drill 2.3) (layers *.Cu *.Mask))
+    (fp_circle (center 0 0) (end 1.15 0) (layer "Edge.Cuts") (width 0.1) (fill none))
   )
-  (footprint "kbd:thread_m2" (layer "F.Cu")
+  (footprint "pica:thread_m2_hole" (layer "F.Cu")
     (at 206.5 86.5)
     (descr "Mounting Hole 2.2mm, no annular, M2")
@@
     (property "Sheetfile" "full.kicad_sch")
     (property "Sheetname" "")
-    (attr exclude_from_pos_files)
+    (attr exclude_from_pos_files exclude_from_bom)
     (fp_text reference "H6" (at -0.95 -0.55) (layer "F.Fab") hide
       (effects (font (size 1 1) (thickness 0.15)))
@@
       (effects (font (size 1 1) (thickness 0.15)))
     )
-    (pad "" np_thru_hole circle locked (at 0 0) (size 2.3 2.3) (drill 2.3) (layers *.Cu *.Mask))
+    (fp_circle (center 0 0) (end 1.15 0) (layer "Edge.Cuts") (width 0.1) (fill none))
   )
-  (footprint "kbd:thread_m2" (layer "F.Cu")
+  (footprint "pica:thread_m2_hole" (layer "F.Cu")
     (at 146 111.5)
     (descr "Mounting Hole 2.2mm, no annular, M2")
@@
       (effects (font (size 1 1) (thickness 0.15)))
     )
-    (pad "" np_thru_hole circle locked (at 0 0) (size 2.3 2.3) (drill 2.3) (layers *.Cu *.Mask))
+    (fp_circle (center 0 0) (end 1.15 0) (layer "Edge.Cuts") (width 0.1) (fill none))
   )
-  (footprint "kbd:thread_m2" (layer "F.Cu")
+  (footprint "pica:thread_m2_hole" (layer "F.Cu")
     (at 197.5 125.5)
     (descr "Mounting Hole 2.2mm, no annular, M2")
@@
       (effects (font (size 1 1) (thickness 0.15)))
     )
-    (pad "" np_thru_hole circle locked (at 0 0) (size 2.3 2.3) (drill 2.3) (layers *.Cu *.Mask))
+    (fp_circle (center 0 0) (end 1.15 0) (layer "Edge.Cuts") (width 0.1) (fill none))
   )
   (gr_line (start 127 126.5) (end 154 135) (layer "Edge.Cuts") (width 0.1))
